Commit message: added the landing platform to obstacle room

File: gym_pybullet_drones/assets/room_w_pad.urdf (robot description, URDF)
Before this commit: robot maze.urdf, 1 links, 0 joints
Links:
- link baseLink: geometry collision mesh filename=room_w_pad.obj scale=1 1 1; visual mesh filename=room_w_pad.obj scale=1 1 1
